Commit message: slam_nav fixes

File: src/yahboomcar_description/urdf/yahboomcar_X3_simple.urdf (robot description, URDF)
Before this commit: robot yahboomcar, 9 links, 8 joints
Joints:
- joint laser_joint: origin xyz=0.0435 0.0001 0.11 rpy=0 0 0 -> xyz=0.0435 0.0001 0.11 rpy=0 0 3.14159

Commit message: Realsense d435i depth replaces Astra. Working.

File: src/yahboomcar_description/urdf/yahboomcar_X3_simple.urdf (robot description, URDF)
Before this commit: robot yahboomcar, 9 links, 8 joints
Links:
- link camera_link: mass None -> 0.01
Joints:
- joint camera_joint: origin xyz=0.057 0.0 0.038 rpy=0 0 0 -> xyz=0.12 0.0 0.0285 rpy=0 0 0

Commit message: URDF adjustments

File: src/yahboomcar_description/urdf/yahboomcar_X3_simple.urdf (robot description, URDF)
Before this commit: robot yahboomcar, 9 links, 8 joints
Links:
- link back_left_wheel: geometry visual cylinder length=0.026 radius=0.032
- link back_right_wheel: geometry visual cylinder length=0.026 radius=0.032
- link base_link: geometry collision box size=0.23 0.15 0.08; visual box size=0.23 0.15 0.08
- link front_left_wheel: geometry visual cylinder length=0.026 radius=0.032
- link front_right_wheel: geometry visual cylinder length=0.026 radius=0.032
- link imu_link: geometry visual box size=0.02 0.025 0.008
Joints:
- joint back_left_joint: origin xyz=-0.06 0.0775 -0.0165 rpy=1.5708 0 0 -> xyz=-0.08 0.087 -0.0495 rpy=1.5708 0 0
- joint back_right_joint: origin xyz=-0.06 -0.0775 -0.0165 rpy=1.5708 0 0 -> xyz=-0.08 -0.087 -0.0495 rpy=1.5708 0 0
- joint base_imu: origin xyz=-0.06 0.01 0.01 rpy=0 3.1415 1.5707 -> xyz=-0.0565 0.015 0.11 rpy=0 3.1415 1.5707
- joint camera_joint: origin xyz=0.12 0.0 0.0285 rpy=0 0 0 -> xyz=0.082 0.0 0.0305 rpy=0 0 0
- joint front_left_joint: origin xyz=0.06 0.0775 -0.0165 rpy=1.5708 0 0 -> xyz=0.08 0.087 -0.0495 rpy=1.5708 0 0
- joint front_right_joint: origin xyz=0.06 -0.0775 -0.0165 rpy=1.5708 0 0 -> xyz=0.08 -0.087 -0.0495 rpy=1.5708 0 0

Commit message: last known good

File: src/yahboomcar_description/urdf/yahboomcar_X3_simple.urdf (robot description, URDF)
Before this commit: robot yahboomcar, 9 links, 8 joints
Joints:
- joint camera_joint: origin xyz=0.082 0.0 0.0305 rpy=0 0 0 -> xyz=0.1 0.0 0.0405 rpy=0 0 0
