Commit message: Remeasured and updated urdf

File: src/yahboomcar_description/urdf/yahboomcar_X3.urdf (robot description, URDF)
Before this commit: robot yahboomcar, 9 links, 8 joints
Links:
- added link camera_tilt_link
- added link camera_tilt_pivot
- link back_left_wheel: mass 0.0515309299357028 -> None; geometry visual cylinder length=0.026 radius=0.032
- link back_right_wheel: mass 0.051540174053366 -> None; geometry visual cylinder length=0.026 radius=0.032
- link base_link: mass 0.486218814966626 -> 0.486; geometry collision box size=0.23 0.15 0.08; visual box size=0.23 0.15 0.08
- link camera_link: mass 0 -> 0.01; geometry visual box size=0.03 0.1 0.03
- link front_left_wheel: mass 0.051543 -> None; geometry visual cylinder length=0.026 radius=0.032
- link front_right_wheel: mass 0.051532 -> None; geometry visual cylinder length=0.026 radius=0.032
- link imu_link: geometry visual box size=0.02 0.025 0.008
- link laser_link: mass 0.0483909504209895 -> None; geometry visual cylinder length=0.04 radius=0.025
Joints:
- removed joint camera_joint
- added joint camera_arm_joint: type fixed, parent camera_tilt_link, child camera_link, origin xyz=0.040 0 0 rpy=0 0 0
- added joint camera_link_to_realsense: type fixed, parent camera_link, child realsense_camera_realsense_camera_link, origin xyz=0 0 0 rpy=0 0 0
- added joint camera_pivot_joint: type fixed, parent base_link, child camera_tilt_pivot, origin xyz=0.089 0.008 0.031 rpy=0 0 0
- added joint camera_tilt_joint: type revolute, parent camera_tilt_pivot, child camera_tilt_link, origin xyz=0 0 0 rpy=0 0 0, axis 0 1 0, limit lower=-0.401 upper=1.204 effort=10.0 velocity=5.0
- joint back_left_joint: limit effort=100 velocity=1 -> (none); origin xyz=-0.08 0.084492 -0.03954 rpy=1.5703 0 0 -> xyz=-0.08 0.087 -0.0495 rpy=1.5708 0 0
- joint back_right_joint: limit effort=100 velocity=1 -> (none); origin xyz=-0.08 -0.0845 -0.03946 rpy=-1.57 0 3.14159 -> xyz=-0.08 -0.087 -0.0495 rpy=1.5708 0 0
- joint base_imu: origin xyz=-0.06 0.01 0.01 rpy=0 3.1415 1.5707 -> xyz=-0.0565 0.015 0.11 rpy=0 3.1415 1.5707
- joint front_left_joint: limit effort=100 velocity=1 -> (none); origin xyz=0.08 0.084492 -0.0389 rpy=1.5703 0 0 -> xyz=0.08 0.087 -0.0495 rpy=1.5708 0 0
- joint front_right_joint: limit effort=100 velocity=1 -> (none); origin xyz=0.08 -0.0845 -0.0389 rpy=-1.5703 0 3.14159 -> xyz=0.08 -0.087 -0.0495 rpy=1.5708 0 0
- joint laser_joint: origin xyz=0.0435 5.25826986680105E-05 0.11 rpy=0 0 0 -> xyz=0.039 0.0 0.082 rpy=0 0 3.14159

Commit message: Camera/servo fixes

File: src/yahboomcar_description/urdf/yahboomcar_X3.urdf (robot description, URDF)
Before this commit: robot yahboomcar, 11 links, 11 joints
Links:
- added link camera_front_marker; visual box size=0.003 0.09 0.025
- added link realsense_camera_realsense_camera_link
- link camera_link: geometry visual box size=0.025 0.09 0.025
Joints:
- added joint camera_front_marker_joint: type fixed, parent camera_link, child camera_front_marker, origin xyz=0.015 0 0 rpy=0 0 0
- joint base_imu: origin xyz=-0.0565 0.015 0.11 rpy=0 3.1415 1.5707 -> xyz=0.0 0.0 0.063 rpy=0 3.1415 1.5707
- joint camera_tilt_joint: axis 0 1 0 -> 0 -1 0
